File: Hardware/Bottom/MusicBox-BOTTOM.brd (EAGLE design)
At the start: 33 x 33 mm, 31 parts, among them U1 AD5242-SO16

Commit message: updates
Parts:
- added J1: (no value), LinnesLab-Connectors:1X07
Connections:
- removed net LED.CTRL: U$4.8
- removed net PPG: C21.2, OP3.1, U1.14
- removed net TIA: C10.2, C15.1, OP4.1, U1.3
- new net A6/TIA: C10.2, C15.1, J1.5, OP4.1, U1.3
- new net A7/PPG: C21.2, J1.7, OP3.1, U1.14
- new net D29/LED.CTRL: J1.6, U$4.8
Changed lines of the file:
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@@
 <attribute name="VALUE" x="5.8928" y="8.3566" size="0.6604" layer="27" rot="R270"/>
+</element>
+<element name="J1" library="LinnesLab-Connectors" package="1X07" value="" x="5" y="33" smashed="yes">
+<attribute name="NAME" x="2.8918" y="36.0734" size="0.6096" layer="25" font="vector" ratio="20"/>
+<attribute name="VALUE" x="3.73" y="30.968" size="0.6096" layer="27" font="vector" ratio="20"/>
 </element>
 </elements>
@@
 <wire x1="15.1892" y1="4.4196" x2="18.4346" y2="11.549" width="0" layer="19" extent="1-1"/>
 </signal>
-<signal name="TIA">
+<signal name="A6/TIA">
 <contactref element="C10" pad="2"/>
 <contactref element="U1" pad="3"/>
 <contactref element="C15" pad="1"/>
 <contactref element="OP4" pad="1"/>
-<wire x1="20.2692" y1="23.6338" x2="12.9692" y2="23.8654" width="0" layer="19" extent="1-1"/>
-<wire x1="24.7904" y1="28.7392" x2="20.2692" y2="23.6338" width="0" layer="19" extent="1-1"/>
-<wire x1="26.2636" y1="10.6934" x2="24.7904" y2="28.7392" width="0" layer="19" extent="1-1"/>
+<contactref element="J1" pad="5"/>
+<wire x1="20.2692" y1="23.6338" x2="24.7904" y2="28.7392" width="0" layer="19" extent="1-1"/>
+<wire x1="12.9692" y1="23.8654" x2="20.2692" y2="23.6338" width="0" layer="19" extent="1-1"/>
+<wire x1="15.16" y1="33" x2="12.9692" y2="23.8654" width="0" layer="19" extent="1-1"/>
+<wire x1="26.2636" y1="10.6934" x2="20.2692" y2="23.6338" width="0" layer="19" extent="1-1"/>
 </signal>
 <signal name="PD.C">
@@
 <wire x1="18.9112" y1="7.112" x2="16.4846" y2="11.549" width="0" layer="19" extent="1-1"/>
 </signal>
-<signal name="LED.CTRL">
+<signal name="D29/LED.CTRL">
 <contactref element="U$4" pad="8"/>
+<contactref element="J1" pad="6"/>
+<wire x1="16.4846" y1="13.9018" x2="17.7" y2="33" width="0" layer="19" extent="1-1"/>
 </signal>
 <signal name="N$10">
@@
 <contactref element="U1" pad="1"/>
 </signal>
-<signal name="PPG">
+<signal name="A7/PPG">
 <contactref element="U1" pad="14"/>
 <contactref element="C21" pad="2"/>
 <contactref element="OP3" pad="1"/>
-<wire x1="32.4104" y1="10.6934" x2="13.4992" y2="9.9314" width="0" layer="19" extent="1-1"/>
-<wire x1="28.134" y1="33.9852" x2="32.4104" y2="10.6934" width="0" layer="19" extent="1-1"/>
+<contactref element="J1" pad="7"/>
+<wire x1="20.24" y1="33" x2="28.134" y2="33.9852" width="0" layer="19" extent="1-1"/>
+<wire x1="32.4104" y1="10.6934" x2="28.134" y2="33.9852" width="0" layer="19" extent="1-1"/>
+<wire x1="13.4992" y1="9.9314" x2="32.4104" y2="10.6934" width="0" layer="19" extent="1-1"/>
 </signal>
 <signal name="N$13">
