File: Hardware/Bottom/MusicBox-BOTTOM.sch (EAGLE design)
At the start: 31 parts, among them U1 AD5242-SO16

Commit message: updates
Parts:
- added J1: (no value), LinnesLab-Connectors:CONN_07
Connections:
- removed net LED.CTRL: U$4.A
- removed net PPG: C21.2, OP3G$1.OUT, U1.B2
- removed net TIA: C10.2, C15.1, OP4G$1.OUT, U1.W1
- new net A6/TIA: C10.2, C15.1, J1.5, OP4G$1.OUT, U1.W1
- new net A7/PPG: C21.2, J1.7, OP3G$1.OUT, U1.B2
- new net D29/LED.CTRL: J1.6, U$4.A
Changed lines of the file:
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@@
 <part name="GND30" library="LinnesLab-Symbols" deviceset="GND" device=""/>
 <part name="SUPPLY24" library="LinnesLab-Symbols" deviceset="3.3V" device=""/>
+<part name="J1" library="LinnesLab-Connectors" deviceset="CONN_07" device=""/>
 </parts>
 <sheets>
@@
 <attribute name="VALUE" x="99.06" y="139.954" size="1.778" layer="96" align="bottom-center"/>
 </instance>
+<instance part="J1" gate="G$1" x="104.14" y="58.42" smashed="yes">
+<attribute name="VALUE" x="99.06" y="48.514" size="1.778" layer="96" font="vector"/>
+<attribute name="NAME" x="99.06" y="71.628" size="1.778" layer="95" font="vector"/>
+</instance>
 </instances>
 <busses>
@@
 </segment>
 </net>
-<net name="TIA" class="0">
+<net name="A6/TIA" class="0">
 <segment>
 <wire x1="-35.56" y1="63.5" x2="-40.64" y2="63.5" width="0.1524" layer="91"/>
@@
 <junction x="-88.9" y="129.54"/>
 </segment>
+<segment>
+<pinref part="J1" gate="G$1" pin="5"/>
+<wire x1="109.22" y1="63.5" x2="111.76" y2="63.5" width="0.1524" layer="91"/>
+<label x="119.38" y="63.5" size="1.778" layer="95"/>
+</segment>
 </net>
 <net name="PD.C" class="0">
@@
 </segment>
 </net>
-<net name="LED.CTRL" class="0">
+<net name="D29/LED.CTRL" class="0">
 <segment>
 <pinref part="U$4" gate="G$1" pin="A"/>
@@
 <wire x1="60.96" y1="66.04" x2="60.96" y2="73.66" width="0.1524" layer="91"/>
 <label x="60.96" y="73.66" size="1.27" layer="95" rot="R180" xref="yes"/>
+</segment>
+<segment>
+<pinref part="J1" gate="G$1" pin="6"/>
+<wire x1="109.22" y1="66.04" x2="111.76" y2="66.04" width="0.1524" layer="91"/>
+<label x="116.84" y="66.04" size="1.778" layer="95"/>
 </segment>
 </net>
@@
 </segment>
 </net>
-<net name="PPG" class="0">
+<net name="A7/PPG" class="0">
 <segment>
 <wire x1="-7.62" y1="63.5" x2="-5.08" y2="63.5" width="0.1524" layer="91"/>
@@
 <label x="50.8" y="121.92" size="1.27" layer="95" xref="yes"/>
 </segment>
-</net>
+<segment>
+<pinref part="J1" gate="G$1" pin="7"/>
+<wire x1="109.22" y1="68.58" x2="111.76" y2="68.58" width="0.1524" layer="91"/>
+<label x="119.38" y="68.58" size="1.778" layer="95"/>
+</segment>
+</net>
