File: Hardware/Top/MusicBox-Top.sch (EAGLE design)
At the start: 51 parts, among them SW1 SWITCH.MOM, SW6 SWITCH.MOM, U2 NRF52832_MODULE_MDBT42, U4 PCF8523

Commit message: updates
Parts:
- added C22: 100n, LinnesLab-Passives:CAPACITOR0603
- added C23, C24: 47p, LinnesLab-Passives:CAPACITOR0603
- added J1: (no value), LinnesLab-Connectors:CONN_07
- added JP2: (no value), LinnesLab-Switches:JUMPER-SMT_2_NO_SILK
- added LED5: RED, LinnesLab-LED:LED0603
- added LED6: YELLOW, LinnesLab-LED:LED0603
- added R1, R2: 0, LinnesLab-Passives:RESISTOR0603
- added R17, R18: 27, LinnesLab-Passives:RESISTOR0603
- added R19, R20: 1k, LinnesLab-Passives:RESISTOR0603
- added U5: FT231XS, LinnesLab-DigitalIC:FT231XS
Connections:
- removed net BATT: R13.1, R14.2
- removed net CD1: SD2.CARD_DETECT
- removed net CHRG.STAT: CHRG2.STAT, R12.1
- removed net CS.OLED: U3./CS
- removed net DC.OLED: U3.DC/I2C_SA0
- removed net RESET.OLED: U3./RES
- removed net RXD: U2.P0.08
- removed net SD.CS: SD2.CS
- removed net SW1: SW1.1, SW6.1
- removed net TXD: U2.P0.06
- new net !CTS: JP2.2, U5.!CTS
- new net A4/BATT: R13.1, R14.2, U2.P0.28/AIN4
- new net A6/TIA: U2.P0.30/AIN6
- new net A7/PPG: U2.P0.31/AIN7
- new net D11/SW1: SW6.1, U2.P0.11
- new net D15/SW2: SW1.1, U2.P0.15
- new net D16/CS.OLED: U2.P0.16, U3./CS
- new net D26/LED.CTRL: U2.P0.29/AIN5
- new net D27/CHRG.STATUS: CHRG2.STAT, R12.1, U2.P0.27
- new net D3/RESET.OLED: U2.P0.03/AIN1, U3./RES
- new net D4/DC.OLED: U2.P0.04/AIN2, U3.DC/I2C_SA0
- new net D5/CD1: SD2.CARD_DETECT, U2.P0.05/AIN3
- new net D7/SD.CS: SD2.CS, U2.P0.07
- new net FT3V3: U5.3V3OUT
- new net N$24: R17.2, U5.USBDM
- new net N$25: R18.2, U5.USBDP
- new net N$26: LED5.C, R19.2
- new net N$27: LED6.C, R20.2
- new net RXD.FT: R2.1, U5.RXD
- new net RXD.NRF: R1.2, U2.P0.08
- new net RXLED: R19.1, U5.CBUS1
- new net TXD.FT: R1.1, U5.TXD
- new net TXD.NRF: R2.2, U2.P0.06
- new net TXLED: R20.1, U5.CBUS2
- net 3.3V: now also C22.2, LED5.A, LED6.A, U5.!RESET, U5.VCCIO
- net DTR: now also U5.!DTR
- net GND: now also C22.1, C23.2, C24.1, JP2.1, U5.GND@16, U5.GND@6
- net SCL: now also R9.1; no longer R8.1
- net SDA: now also R8.1; no longer R9.1
- net USB+: now also C23.1, R18.1
- net USB-: now also C24.2, R17.1
- net V_USB: now also U5.VCC
Other:
- note added: "I don't remember if CTS needs to be grounded or left floating so here's a jumper to ground so it can be configued either way dynamically."
- note added: "TXD goes to RX on the other device RXD goes to TX on the other device"
- moved on the sheet: R8, R9
